File: hardware/Bats-n-Gons2.brd (EAGLE design)
At the start: 59.4 x 53.3 mm, 69 parts, among them SW1 SMD_SWITCH, U1 SAMD51PXXA, U2 IS31AP4991, X1 32.768

Commit message: DRC checks out
Routing:
- net PA21: track 32.7 -> 6.18 mm, vias 1 -> 0
- net D11: track 24.9 -> 0.00 mm
- net D0: track 24.5 -> 0.00 mm, vias 2 -> 0
- net PA22: track 33.6 -> 10.3 mm, vias 1 -> 0
- net PA23: track 31.0 -> 9.67 mm, vias 2 -> 0
- net D1: track 21.3 -> 0.00 mm, vias 2 -> 0
- net D10: track 20.5 -> 0.00 mm
- net +3.3V: track 157.2 -> 143.9 mm, vias 24 -> 21
- net PA20: track 35.6 -> 22.9 mm
- net N$6: track 8.31 -> 0.00 mm
- net GND: track 3.29 -> 1.43 mm, vias 64 -> 60
- net +5V: track 59.8 -> 58.6 mm
- net NEOPIX: track 18.1 -> 17.1 mm
